File: KICAD/MPD.sch (KiCad schematic (older format))
At the start: 1 part

Commit message: working on schematic (version 1.1)
Parts:
- added C? (x5): CP, symbol CP
- added C? (x8): C, symbol C
- added D? (x17): D, symbol D
- added D? (x4): D_Zener, symbol D_Zener
- added R? (x44): R, symbol R
- added U? (x6): LM2904, symbol LM2904
Connections:
- new net: R?.1, R?.2 (x6)
- new net: D?.1 (K), R?.2 (x6)
- new net: D?.2 (A), R?.1, R?.1 (x3)
- new net: C?.1, D?.1 (K), R?.1, U?.3 (+) (x3)
- new net: C?.1, R?.1, R?.2, U?.1 (x3)
- new net: C?.2, R?.2, U?.2 (-) (x3)
- new net: D?.1 (K), R?.1, R?.2 (x3)
- new net: R?.1, R?.1 (x3)
- new net: R?.2, R?.2 (x3)
- new net: C?.2, R?.1
- new net: C?.1, D?.1 (K), D?.2 (A)
- new net: C?.1, D?.1 (K), R?.2
- new net +5V: C?.1, C?.1, D?.1 (K), R?.1, R?.1, R?.1, R?.1
- new net ADC0: C?.1, R?.1
- new net ADC1: C?.1, R?.1
- new net ADC2: C?.1, R?.1
- new net GNDREF: C?.2, C?.2, C?.2, C?.2, C?.2, C?.2, C?.2, C?.2, C?.2, D?.2 (A), D?.2 (A), D?.2 (A), D?.2 (A), D?.2 (A), R?.2, R?.2, R?.2, R?.2, R?.2, R?.2, R?.2, R?.2, R?.2
- new net INT0: R?.1, R?.2
- new net INT1: R?.1, R?.2
- new net INT2: R?.1, R?.2
- new net INT3: R?.1, U?.1
- new net INT4: R?.1, U?.1
- new net INT5: R?.1, U?.1
- new net PHASE_A: D?.2 (A), D?.2 (A), R?.2
- new net PHASE_B: D?.2 (A), D?.2 (A)
- new net PHASE_C: D?.2 (A), D?.2 (A)
- new net TCA_A: D?.1 (K), D?.2 (A), R?.2, U?.3 (+)
- new net TCA_B: D?.1 (K), D?.2 (A), R?.1, U?.2 (-)
- new net TCB_A: D?.1 (K), D?.2 (A), R?.2, U?.3 (+)
- new net TCB_B: D?.1 (K), D?.2 (A), R?.1, U?.2 (-)
- new net TCC_A: D?.1 (K), D?.2 (A), R?.2, U?.3 (+)
- new net TCC_B: D?.1 (K), D?.2 (A), R?.1, U?.2 (-)
Other:
- note added: "AC/PULSE voltage converter unit\n(top side)"
- note added: "current sensor to pulse voltage converter unit\n(top side)\n"
- note added: "power supply unit \n(bottom side)"
- note added: "voltage measuring unit\n(top side)"
- moved on the sheet: U?

Commit message: update schematic
Parts:
- removed U? (x3): LM2904, symbol LM2904
- added C? (x5): C, symbol C
- added D?: Q_TRIAC_A1A2G, symbol Q_TRIAC_A1A2G
- added P?: CONN_01X04, symbol CONN_01X04
- added R? (x8): R, symbol R
- added U? (x3): LM2904, symbol LM2904
- added U?: MOC3023M, DIP-6, symbol MOC3023M
- added U?: LM1117-3.3, symbol LM1117-3.3
- added Y?: Crystal, symbol Crystal
Connections:
- net labels added: +3.3V, ADC3, DATA_RX, DATA_TX, FREQ_A, FREQ_B, FREQ_C, GND, OCS_IN, OSC_IN, OSC_OUT, STARTER_CONTROL, STARTER_POWER, SWCLK, SWDIO, TRIAC_CONTROL
- wire segments 164 -> 239
Other:
- note added: "MCU unit <stm32f030c8t6 for 1.1 version> \n(top side)"
- note added: "programming interface (SWD only)"
- note added: "starter control unit\n(bottom side)"
- moved on the sheet: C?, D?, R?, U?, U?A

Commit message: finished schematic for alfa version
Parts:
- removed C? (x2): C, symbol C
- removed U?: LM1117-3.3, symbol LM1117-3.3
- added C19, C20: 22n, symbol C
- added C4: 4u7, symbol CP
- added C5: 1u, symbol CP
- added C6, C7: 100n, symbol C
- added C8: 10n, symbol C
- added C9: 10u, symbol CP
- added D21: IR, symbol LED_Small
- added D7, D8: LED, symbol LED
- added F1, F2: Fuse, symbol Fuse
- added J1: Screw_Terminal_1x04, symbol Screw_Terminal_1x04
- added J2: Screw_Terminal_1x06, symbol Screw_Terminal_1x06
- added J3, J4, J5: Screw_Terminal_1x02, symbol Screw_Terminal_1x02
- added P2, P4: CONN_01X02, symbol CONN_01X02
- added P3: CONN_01X04, symbol CONN_01X04
- added P5: CONN_01X03, symbol CONN_01X03
- added Q1: Q_NPN_CBE, symbol Q_NPN_CBE
- added R13, R14: 330R, symbol R
- added R29, R31, R34: 220R, symbol R
- added R53: 10R, symbol R
- added R54: 1k5, symbol R
- added R55, R56: 1k, symbol R
- added R57: 220, symbol R
- added R58: 220k, symbol R
- added U2: AMS1117-3.3, Package_TO_SOT_SMD:SOT-223-3_TabPin2, symbol AMS1117-3.3
- added U6: LM2904, symbol LM2904
- C1, C11, C14: renamed from C?; value CP -> 1u
- C10: renamed from C?; value C -> 1n
- C12, C13, C15, C16, C2, C3: renamed from C?; value C -> 22n
- C17, C18: renamed from C?; value C -> 20p
- C21: renamed from C?; value C -> 2u2 x 400V
- C22, C23: renamed from C?; value CP -> 100u x 25V
- C24: renamed from C?; value C -> 100n
- D1, D10, D13, D17, D19, D2, D22, D23, D5, D6, D9: renamed from D?; value D -> 1A7
- D11, D12, D15, D16, D3, D4: renamed from D?; value D -> SM4001
- D14, D18, D20: renamed from D?; value D_Zener -> BXV5C5v1
- D24: renamed from D?; value D_Zener -> 1N4733A
- R1, R23, R9: renamed from R?; value R -> 220k
- R10, R2, R24: renamed from R?; value R -> 110k
- R11, R12, R16, R17, R21, R22, R32, R33, R38, R4, R44, R45, R7: renamed from R?; value R -> 10k
- R15, R25, R3: renamed from R?; value R -> 1k
- R18, R26, R5: renamed from R?; value R -> 3k3
- R19, R27, R6: renamed from R?; value R -> 100k
- R20, R28, R8: renamed from R?; value R -> 220
- R30: renamed from R?; value R -> 390R
- R35, R36, R41, R42, R48, R49: renamed from R?; value R -> 1k8
- R37, R39, R40, R43, R46, R47, R50, R51, R52: renamed from R?; value R -> 1k5
- R59: renamed from R?; value R -> 10R
- R60: renamed from R?; value R -> 510R
- R61: renamed from R?; value R -> 330R
- R62, R63: renamed from R?; value R -> 320R
- Y1: renamed from Y?; value Crystal -> 8 Mhz
- gave numbers to parts that had none: 7
Connections:
- net labels added: +3V3, CP_A, CP_B, CP_C, LED_GREEN, LED_RED, POWER, TEMP, TEMP_SENSOR
- net labels removed: ADC3, OCS_IN
- wire segments 239 -> 339
- no-connect marks 0 -> 17
Other:
- note added: "irDA unit for data transmit and programming"
- note added: "programmable temperature sensor(thermistor)\n"
- moved on the sheet: C10, C17, C18, C21, C22, C23, C24, D22, D23, D24, P1, R11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

Commit message: fix mcu unit
Parts:
- removed C21: 2u2 x 400V, symbol C
- removed C22, C23: 100u x 25V, symbol CP
- removed C24: 100n, symbol C
- removed D22, D23: 1A7, symbol D
- removed D24: 1N4733A, symbol D_Zener
- removed D25: Q_TRIAC_A1A2G, symbol Q_TRIAC_A1A2G
- removed F1, F2: Fuse, symbol Fuse
- removed J1: Screw_Terminal_1x04, symbol Screw_Terminal_1x04
- removed J2: Screw_Terminal_1x06, symbol Screw_Terminal_1x06
- removed J3, J4, J5: Screw_Terminal_1x02, symbol Screw_Terminal_1x02
- removed P3: CONN_01X04, symbol CONN_01X04
- removed P4: CONN_01X02, symbol CONN_01X02
- removed R58: 220k, symbol R
- removed R59: 10R, symbol R
- removed R60: 510R, symbol R
- removed R61: 330R, symbol R
- removed R62, R63: 320R, symbol R
- removed U6: LM2904, symbol LM2904
- removed U7: MOC3023M, DIP-6, symbol MOC3023M
- added C?: 10u, symbol CP
- added D? (x2): D, symbol D
- added P?: CONN_01X03, symbol CONN_01X03
- added Q? (x2): Q_NMOS_GDS, symbol Q_NMOS_GDS
- added Q?: Q_NPN_BEC, symbol Q_NPN_BEC
- added Q?: Q_PNP_BCE, symbol Q_PNP_BCE
- added R? (x5): R, symbol R
- added U? (x4): LM2904, symbol LM2904
- added U?: AMS1117-5.0, Package_TO_SOT_SMD:SOT-223-3_TabPin2, symbol AMS1117-5.0
- renumbered C1 to C?, C11 to C?, C14 to C?, C13 to C?, C3 to C?, C16 to C?, C2 to C?, C15 to C?, C12 to C?, C10 to C?, C17 to C?, C18 to C?, C20 to C?, C19 to C?, C6 to C?, C4 to C?, C5 to C?, C7 to C?, C8 to C?, C9 to C?, D1 to D?, D2 to D?, D5 to D?, D6 to D?, D9 to D?, D10 to D?, D14 to D?, D13 to D?, D18 to D?, D17 to D?, D20 to D?, D19 to D?, D3 to D?, D4 to D?, D11 to D?, D12 to D?, D15 to D?, D16 to D?, D7 to D?, D8 to D?, D21 to D?, P1 to P?, P5 to P?, P2 to P?, Q1 to Q?, R1 to R?, R2 to R?, R5 to R?, R6 to R?, R3 to R?, R8 to R?, R9 to R?, R10 to R?, R18 to R?, R19 to R?, R15 to R?, R20 to R?, R23 to R?, R24 to R?, R26 to R?, R27 to R?, R25 to R?, R28 to R?, R35 to R?, R36 to R?, R37 to R?, R39 to R?, R40 to R?, R41 to R?, R42 to R?, R43 to R?, R46 to R?, R47 to R?, R48 to R?, R49 to R?, R50 to R?, R51 to R?, R52 to R?, R4 to R?, R7 to R?, R16 to R?, R17 to R?, R22 to R?, R32 to R?, R33 to R?, R38 to R?, R44 to R?, R45 to R?, R30 to R?, R21 to R?, R11 to R?, R12 to R?, R29 to R?, R31 to R?, R34 to R?, R13 to R?, R14 to R?, R56 to R?, R57 to R?, R53 to R?, R55 to R?, R54 to R?, U4 to U?, U1 to U?, U3 to U?, U5 to U?, U2 to U?, Y1 to Y?
Connections:
- net labels added: +12V, MOTOR_PHASE_A, MOTOR_PHASE_B, SCL, SDA, TEMP_CONTROL
- net labels removed: POWER, STARTER_CONTROL, STARTER_POWER
- wire segments 339 -> 318
Other:
- note added: "I2C bus(for LCD connector)"
- note removed: "power supply unit \n(bottom side)"
- note removed: "starter control unit\n(bottom side)"
- moved on the sheet: C?, D?, P?, Q?, R?, U?, Y?

Commit message: KiCAD version 5.0 fix schematics
Parts:
- removed P?: CONN_01X02, symbol CONN_01X02
- removed P?: CONN_01X03, symbol CONN_01X03
- removed Q?: Q_PNP_BCE, symbol Q_PNP_BCE
- added J1: Conn_01x03_Female, symbol Connector:Conn_01x03_Female
- added J2, J5, J6, J7: Conn_01x02_Female, symbol Connector:Conn_01x02_Female
- added J3: Conn_01x06_Female, symbol Connector:Conn_01x06_Female
- added J4: Conn_01x04_Female, symbol Connector:Conn_01x04_Female
- added Q2: Q_PNP_BEC, symbol Device:Q_PNP_BEC
- C1, C13, C14, C15, C2, C5, C7: renamed from C?; symbol CP -> Device:CP
- C10, C11, C12, C16, C17, C18, C19, C20, C21, C3, C4, C6, C8, C9: renamed from C?; symbol C -> Device:C
- D1, D10, D11, D12, D13, D14, D18, D19, D2, D20, D21, D22, D23, D6, D7, D8, D9: renamed from D?; symbol D -> Device:D
- D15, D16, D17: renamed from D?; symbol D_Zener -> Device:D_Zener
- D3: renamed from D?; symbol LED_Small -> Device:LED_Small
- D4, D5: renamed from D?; symbol LED -> Device:LED
- P1: renamed from P?; symbol CONN_01X03 -> MPD-rescue:CONN_01X03
- P2: renamed from P?; symbol CONN_01X04 -> MPD-rescue:CONN_01X04
- Q1: renamed from Q?; symbol Q_NPN_BEC -> Device:Q_NPN_BEC
- Q3, Q4: renamed from Q?; symbol Q_NMOS_GDS -> Device:Q_NMOS_GDS
- Q5: renamed from Q?; symbol Q_NPN_CBE -> Device:Q_NPN_CBE
- R1, R10, R11, R12, R13, R14, R15, R16, R17, R18, R19, R2, R20, R21, R22, R23, R24, R25, R26, R27, R28, R29, R3, R30, R31, R32, R33, R34, R35, R36, R37, R38, R39, R4, R40, R41, R42, R43, R44, R45, R46, R47, R48, R49, R5, R50, R51, R52, R53, R54, R55, R56, R57, R58, R59, R6, R60, R61, R62, R7, R8, R9: renamed from R?; symbol R -> Device:R
- U1: renamed from U?; symbol AMS1117-5.0 -> Regulator_Linear:AMS1117-5.0
- U2: renamed from U?; symbol AMS1117-3.3 -> Regulator_Linear:AMS1117-3.3
- U3, U5, U6, U7: renamed from U?; symbol LM2904 -> Amplifier_Operational:LM2904
- U4: renamed from U?; symbol STM32F030C8Tx -> MCU_ST_STM32F0:STM32F030C8Tx
- Y1: renamed from Y?; symbol Crystal -> Device:Crystal
Connections:
- net GNDREF is gone; now on net GND: C19.2, C20.2, C21.2
- net +12V: now also J2.2 (Pin_2)
- net +3V3: now also J4.4 (Pin_4)
- net +5V: now also U3.8 (V+), U5.8 (V+), U6.8 (V+)
- net GND: now also J2.1 (Pin_1), J4.1 (Pin_1), J7.1 (Pin_1), Q2.2 (E)
- net INT1: now also R17.2
- net INT2: now also R18.2
- net MOTOR_PHASE_A: now also J6.2 (Pin_2)
- net MOTOR_PHASE_B: now also J6.1 (Pin_1)
- net PHASE_A: now also J1.3 (Pin_3)
- net PHASE_B: now also J1.2 (Pin_2)
- net PHASE_C: now also J1.1 (Pin_1)
- net SCL: now also U4.42 (PB6), J5.1 (Pin_1)
- net SDA: now also U4.43 (PB7), J5.2 (Pin_2)
- net SWCLK: now also J4.2 (Pin_2)
- net SWDIO: now also J4.3 (Pin_3)
- net TCA_A: now also J3.6 (Pin_6)
- net TCA_B: now also J3.5 (Pin_5)
- net TCB_A: now also J3.4 (Pin_4)
- net TCB_B: now also J3.3 (Pin_3)
- net TCC_A: now also J3.2 (Pin_2)
- net TCC_B: now also J3.1 (Pin_1)
- net TEMP_CONTROL: now also U4.29 (PA8)
- net TRIAC_CONTROL: now also J7.2 (Pin_2)
- net at Q1.2 (E), Q3.1 (G), Q4.1 (G): now also Q2.3 (C)
- net at Q1.1 (B), R1.1: now also Q2.1 (B)
- no-connect marks 17 -> 14
Other:
- moved on the sheet: C3, C6, D1, D2, Q1, R1, R2, R3, R4, R5, U3B

Commit message: -pcb finished
Parts:
- removed D11, D13, D14: 1A7, symbol Device:D
- removed J4: Conn_01x04_Female, symbol Connector:Conn_01x04_Female
- removed P1: CONN_01X03, symbol MPD-rescue:CONN_01X03
- removed P2: CONN_01X04, symbol MPD-rescue:CONN_01X04
- removed unit 2 of U3
- added J2: Conn_01x02_Female, Connector_PinHeader_2.54mm:PinHeader_1x02_P2.54mm_Vertical, symbol Connector:Conn_01x02_Female
- added J7: Conn_01x03_Female, Connector_PinHeader_2.54mm:PinHeader_1x03_P2.54mm_Vertical, symbol Connector:Conn_01x03_Female
- added J8: Conn_01x04_Female, Connector_PinHeader_2.54mm:PinHeader_1x04_P2.54mm_Vertical, symbol Connector:Conn_01x04_Female
- added unit 3 of U4
- added unit 1 of U7
- C1, C2: footprint (none) -> Capacitor_SMD:CP_Elec_6.3x5.4
- C10, C11, C12, C16, C17, C18, C19, C20, C21, C3, C4, C6, C8, C9: footprint (none) -> Capacitor_SMD:C_1206_3216Metric_Pad1.42x1.75mm_HandSolder
- C13, C14, C15, C5, C7: footprint (none) -> Capacitor_SMD:CP_Elec_4x5.4
- D1, D2: footprint (none) -> Diode_SMD:D_SMB
- D10, D9: footprint (none) -> Diode_SMD:D_SMA
- D11: renamed from D12; footprint (none) -> Diode_SMD:D_SMA
- D12: renamed from D15; footprint (none) -> Diode_THT:D_DO-41_SOD81_P2.54mm_Vertical_AnodeUp
- D13: renamed from D16; footprint (none) -> Diode_THT:D_DO-41_SOD81_P2.54mm_Vertical_AnodeUp
- D14: renamed from D17; footprint (none) -> Diode_THT:D_DO-41_SOD81_P2.54mm_Vertical_AnodeUp
- D15: renamed from D18; footprint (none) -> Diode_SMD:D_SMA
- D16: renamed from D19; footprint (none) -> Diode_SMD:D_SMA
- D17: renamed from D20; footprint (none) -> Diode_SMD:D_SMA
- D18: renamed from D21; footprint (none) -> Diode_SMD:D_SMA
- D19: renamed from D22; footprint (none) -> Diode_SMD:D_SMA
- D20: renamed from D23; footprint (none) -> Diode_SMD:D_SMA
- D3: footprint (none) -> LED_THT:LED_D5.0mm
- D4, D5: footprint (none) -> LED_SMD:LED_0805_2012Metric
- D6, D7, D8: footprint (none) -> Diode_THT:D_DO-41_SOD81_P2.54mm_Vertical_AnodeUp
- J1: renamed from J6; footprint (none) -> Connector_PinHeader_2.54mm:PinHeader_1x02_P2.54mm_Vertical
- J3: renamed from J2; footprint (none) -> Connector_PinHeader_2.54mm:PinHeader_1x02_P2.54mm_Vertical
- J4: renamed from J1; footprint (none) -> Connector_PinHeader_2.54mm:PinHeader_1x03_P2.54mm_Vertical
- J5: footprint (none) -> Connector_PinHeader_2.54mm:PinHeader_1x02_P2.54mm_Vertical
- J6: renamed from J3; footprint (none) -> Connector_PinHeader_2.54mm:PinHeader_1x06_P2.54mm_Vertical
- J9: renamed from J7; footprint (none) -> Connector_PinHeader_2.54mm:PinHeader_1x02_P2.54mm_Vertical
- Q1, Q2, Q5: footprint (none) -> Package_TO_SOT_SMD:SOT-23
- Q3, Q4: footprint (none) -> Package_TO_SOT_SMD:SOT-223-3_TabPin2
- R1, R10, R11, R12, R13, R14, R15, R16, R17, R18, R19, R2, R20, R21, R22, R23, R24, R25, R26, R27, R28, R29, R3, R30, R31, R32, R33, R34, R35, R36, R37, R38, R39, R4, R40, R41, R42, R43, R44, R45, R46, R47, R48, R49, R5, R50, R51, R52, R53, R54, R55, R56, R57, R58, R59, R6, R60, R61, R62, R7, R8, R9: footprint (none) -> Resistor_SMD:R_1206_3216Metric_Pad1.42x1.75mm_HandSolder
- U4, U6: renamed from U5; footprint (none) -> Package_SO:Zetex_SM8
- U5: renamed from U3; footprint (none) -> Package_SO:Zetex_SM8
- U5: renamed from U7; footprint (none) -> Package_SO:Zetex_SM8
- U6: footprint (none) -> Package_SO:Zetex_SM8
- U7: renamed from U6; footprint (none) -> Package_SO:Zetex_SM8
- Y1: footprint (none) -> Crystal:Crystal_SMD_HC49-SD
- renumbered U4 to U3
Connections:
- net +3V3: now also J8.4 (Pin_4)
- net +5V: now also R14.1, R15.1, J2.2 (Pin_2), J7.3 (Pin_3), U4.8 (V+)
- net CP_A: now also D8.1 (K), R23.2, R31.2; no longer D11.2 (A), R26.1, R29.1
- net CP_B: now also D6.1 (K), R21.2, R32.2; no longer D9.2 (A), R24.1, R27.1
- net CP_C: now also D7.1 (K), R22.2, R30.2; no longer D10.2 (A), R25.1, R28.1
- net DATA_RX: now also J7.2 (Pin_2)
- net GND: now also Q2.3 (C), J2.1 (Pin_1), J7.1 (Pin_1), J8.1 (Pin_1), U4.4 (V-); no longer Q2.2 (E)
- net SWCLK: now also J8.2 (Pin_2)
- net SWDIO: now also J8.3 (Pin_3)
- net at C3.1, R4.1, R5.2: now also U7.1
- net at C3.2, R4.2: now also U7.2 (-)
- net at Q1.2 (E), Q3.1 (G), Q4.1 (G): now also Q2.2 (E); no longer Q2.3 (C)
- net at D1.2 (A), R3.1: now also U7.3 (+)
- new net: D11.2 (A), R26.1, R29.1
- new net: D9.2 (A), R24.1, R27.1
- new net: D10.2 (A), R25.1, R28.1
Other:
- moved on the sheet: J5
