File: KICAD/MPD.kicad_pcb (KiCad board)
At the start: 2 copper layers, 69.8 x 69.9 mm, 125 parts, among them J1 Conn_01x02_Female, J2 Conn_01x02_Female, J3 Conn_01x02_Female, J4 Conn_01x03_Female, J5 Conn_01x02_Female, J6 Conn_01x06_Female, J7 Conn_01x03_Female, J8 Conn_01x04_Female, J9 Conn_01x02_Female, Q1 Q_NPN_BEC, Q2 Q_PNP_BEC, Q3 Q_NMOS_GDS, Q4 Q_NMOS_GDS, Q5 Q_NPN_CBE, U1 AMS1117-5.0, U2 AMS1117-3.3, U3 STM32F030C8Tx, U4 LM2904, U5 LM2904, U6 LM2904, U7 LM2904, Y1 8 Mhz

Commit message: MPD rev.A0 released
Other:
- board text added: "*var*"
- board text added: "+12V"
- board text added: "5V"
- board text added: "A"
- board text added: "B"
- board text added: "C"
- board text added: "CA"
- board text added: "CB"
- board text added: "CC"
- board text added: "GND"
- board text added: "I2C"
- board text added: "IrDA"
- board text added: "MPD rev. A.0"
- board text added: "actuator"
- board text added: "temp"
- board text removed: "***"
- board text removed: "MPD rev. 1.0"
